Commit message: initial commit

File: hal_rrbot_control/urdf/hal_rrbot_gripper.xacro (robot description, xacro)
@@ -42,20 +42,20 @@
     <link name="${prefix}gripper_base">
       <collision>
-	<origin xyz="0 0 ${base_h/2}" rpy="0 0 0"/>
-	<geometry>
-	  <box size="${base_w} ${d} ${base_h}"/>
-	</geometry>
+        <origin xyz="0 0 ${base_h/2}" rpy="0 0 0"/>
+        <geometry>
+          <box size="${base_w} ${d} ${base_h}"/>
+        </geometry>
       </collision>
       <visual>
-	<origin xyz="0 0 ${base_h/2}" rpy="0 0 0"/>
-	<geometry>
-	  <box size="${base_w} ${d} ${base_h}"/>
-	</geometry>
+        <origin xyz="0 0 ${base_h/2}" rpy="0 0 0"/>
+        <geometry>
+          <box size="${base_w} ${d} ${base_h}"/>
+        </geometry>
         <material name="red"/>
       </visual>
       <inertial>
-	<origin xyz="0 0 ${base_h/2}" rpy="0 0 0"/>
-	<mass value="${base_mass}"/>
-	<inertia
+        <origin xyz="0 0 ${base_h/2}" rpy="0 0 0"/>
+        <mass value="${base_mass}"/>
+        <inertia
 	    ixx="${base_mass/12.0 * (d**2 + base_h**2)}" ixy="0.0" ixz="0.0"
 	    iyy="${base_mass/12.0 * (base_w**2 + base_h**2)}" iyz="0.0"
@@ -65,20 +65,20 @@
     <link name="${prefix}gripper_finger_link1">
       <collision>
-	<origin xyz="0 0 ${finger_h/2}" rpy="0 0 0"/>
-	<geometry>
-	  <box size="${finger_w} ${d} ${finger_h}"/>
-	</geometry>
+        <origin xyz="0 0 ${finger_h/2}" rpy="0 0 0"/>
+        <geometry>
+          <box size="${finger_w} ${d} ${finger_h}"/>
+        </geometry>
       </collision>
       <visual>
-	<origin xyz="0 0 ${finger_h/2}" rpy="0 0 0"/>
-	<geometry>
-	  <box size="${finger_w} ${d} ${finger_h}"/>
-	</geometry>
+        <origin xyz="0 0 ${finger_h/2}" rpy="0 0 0"/>
+        <geometry>
+          <box size="${finger_w} ${d} ${finger_h}"/>
+        </geometry>
         <material name="red"/>
       </visual>
       <inertial>
-	<origin xyz="0 0 ${finger_h/2}" rpy="0 0 0"/>
-	<mass value="${finger_mass}"/>
-	<inertia
+        <origin xyz="0 0 ${finger_h/2}" rpy="0 0 0"/>
+        <mass value="${finger_mass}"/>
+        <inertia
 	    ixx="${finger_mass/12.0 * (d**2 + finger_h**2)}" ixy="0.0" ixz="0.0"
 	    iyy="${finger_mass/12.0 * (finger_w**2 + finger_h**2)}" iyz="0.0"
@@ -88,20 +88,20 @@
     <link name="${prefix}gripper_finger_link2">
       <collision>
-	<origin xyz="0 0 ${finger_h/2}" rpy="0 0 0"/>
-	<geometry>
-	  <box size="${finger_w} ${d} ${finger_h}"/>
-	</geometry>
+        <origin xyz="0 0 ${finger_h/2}" rpy="0 0 0"/>
+        <geometry>
+          <box size="${finger_w} ${d} ${finger_h}"/>
+        </geometry>
       </collision>
       <visual>
-	<origin xyz="0 0 ${finger_h/2}" rpy="0 0 0"/>
-	<geometry>
-	  <box size="${finger_w} ${d} ${finger_h}"/>
-	</geometry>
+        <origin xyz="0 0 ${finger_h/2}" rpy="0 0 0"/>
+        <geometry>
+          <box size="${finger_w} ${d} ${finger_h}"/>
+        </geometry>
         <material name="red"/>
       </visual>
       <inertial>
-	<origin xyz="0 0 0" rpy="0 0 0"/>
-	<mass value="${finger_mass}"/>
-	<inertia
+        <origin xyz="0 0 0" rpy="0 0 0"/>
+        <mass value="${finger_mass}"/>
+        <inertia
 	    ixx="${finger_mass/12.0 * (d**2 + finger_h**2)}" ixy="0.0" ixz="0.0"
 	    iyy="${finger_mass/12.0 * (finger_w**2 + finger_h**2)}" iyz="0.0"

File: interruptible_joint_trajectory_controller/test/rrbot.xacro (robot description, xacro)
@@ -4,10 +4,16 @@
   <!-- Constants for robot dimensions -->
   <xacro:property name="PI" value="3.1415926535897931"/>
-  <xacro:property name="width" value="0.1" /> <!-- Square dimensions (widthxwidth) of beams -->
-  <xacro:property name="height1" value="2" /> <!-- Link 1 -->
-  <xacro:property name="height2" value="1" /> <!-- Link 2 -->
-  <xacro:property name="height3" value="1" /> <!-- Link 3 -->
-  <xacro:property name="camera_link" value="0.05" /> <!-- Size of square 'camera' box -->
-  <xacro:property name="axel_offset" value="0.05" /> <!-- Space btw top of beam and the each joint -->
+  <xacro:property name="width" value="0.1" />
+  <!-- Square dimensions (widthxwidth) of beams -->
+  <xacro:property name="height1" value="2" />
+  <!-- Link 1 -->
+  <xacro:property name="height2" value="1" />
+  <!-- Link 2 -->
+  <xacro:property name="height3" value="1" />
+  <!-- Link 3 -->
+  <xacro:property name="camera_link" value="0.05" />
+  <!-- Size of square 'camera' box -->
+  <xacro:property name="axel_offset" value="0.05" />
+  <!-- Space btw top of beam and the each joint -->
   <material name="black">
     <color rgba="0.0 0.0 0.0 1.0"/>
@@ -27,5 +33,5 @@
       <origin xyz="0 0 ${height1/2}" rpy="0 0 0"/>
       <geometry>
-  <box size="${width} ${width} ${height1}"/>
+        <box size="${width} ${width} ${height1}"/>
       </geometry>
     </collision>
@@ -33,5 +39,5 @@
       <origin xyz="0 0 ${height1/2}" rpy="0 0 0"/>
       <geometry>
-  <box size="${width} ${width} ${height1}"/>
+        <box size="${width} ${width} ${height1}"/>
       </geometry>
       <material name="orange"/>
@@ -59,5 +65,5 @@
       <origin xyz="0 0 ${height2/2 - axel_offset}" rpy="0 0 0"/>
       <geometry>
-  <box size="${width} ${width} ${height2}"/>
+        <box size="${width} ${width} ${height2}"/>
       </geometry>
     </collision>
@@ -65,5 +71,5 @@
       <origin xyz="0 0 ${height2/2 - axel_offset}" rpy="0 0 0"/>
       <geometry>
-  <box size="${width} ${width} ${height2}"/>
+        <box size="${width} ${width} ${height2}"/>
       </geometry>
       <material name="black"/>
@@ -91,5 +97,5 @@
       <origin xyz="0 0 ${height3/2 - axel_offset}" rpy="0 0 0"/>
       <geometry>
-  <box size="${width} ${width} ${height3}"/>
+        <box size="${width} ${width} ${height3}"/>
       </geometry>
     </collision>
@@ -97,5 +103,5 @@
       <origin xyz="0 0 ${height3/2 - axel_offset}" rpy="0 0 0"/>
       <geometry>
-  <box size="${width} ${width} ${height3}"/>
+        <box size="${width} ${width} ${height3}"/>
       </geometry>
       <material name="orange"/>
